Commit message: Modified README, improved visualization of the robot in gazebo and now rviz starts automatically with the correct configuration (slam or amcl)

File: ros_ws/src/bumperbot_description/urdf/bumperbot.urdf.xacro (robot description, xacro)
@@ -42,4 +42,5 @@
                 <mesh filename="package://bumperbot_description/meshes/base_link.STL"/>
             </geometry>
+            <material name="light_grey"/>
         </visual>
         <!-- Ora iniziamo a inserire i parametri utili a gazebo per la simulazione. Gli dico che l'hitbox è la stessa
@@ -77,4 +78,5 @@
                 <mesh filename="package://bumperbot_description/meshes/wheel_right_link.STL"/>
             </geometry>
+            <material name="black"/>
         </visual>
         <!-- In questo caso il file STL della ruota che uso è molto complesso(la mesh è piena di superfici piccole)
@@ -109,4 +111,5 @@
                 <mesh filename="package://bumperbot_description/meshes/wheel_left_link.STL"/>
             </geometry>
+            <material name="black"/>
         </visual>
         <!-- Roba per la simulazione-->
@@ -139,4 +142,5 @@
                 <mesh filename="package://bumperbot_description/meshes/caster_front_link.STL"/>
             </geometry>
+            <material name="red"/>
         </visual>
         <collision>
@@ -166,4 +170,5 @@
                 <mesh filename="package://bumperbot_description/meshes/caster_rear_link.STL"/>
             </geometry>
+            <material name="red"/>
         </visual>
         <collision>
@@ -193,7 +198,5 @@
         <mesh filename="package://bumperbot_description/meshes/imu_link.STL" />
       </geometry>
-      <material name="">
-        <color rgba="0.792156862745098 0.819607843137255 0.933333333333333 1" />
-      </material>
+       <material name="blue"/>
     </visual>
     <collision>
@@ -219,8 +222,9 @@
     </inertial>
     <visual>
-      <origin xyz="0 0 0" rpy="0 0 0" />
+      <origin xyz="0 0 0" rpy="0 0 3.14" />
       <geometry>
         <mesh filename="package://bumperbot_description/meshes/laser_link.STL" />
       </geometry>
+      <material name="black"/>
     </visual>
     <collision>
@@ -237,3 +241,21 @@
     <axis xyz="0 0 0" />
   </joint>
+  <material name="blue">
+    <color rgba="0 0 1 1"/>
+  </material>
+  <material name="black">
+    <color rgba="0.03 0.03 0.03 1"/>
+  </material>
+  <material name="silver">
+    <color rgba="0.79 0.82 0.93 1"/>
+  </material>
+  <material name="dark_grey">
+    <color rgba="0.2 0.2 0.2 1"/>
+  </material>
+  <material name="red">
+    <color rgba="1 0 0 1"/>
+  </material>
+  <material name="light_grey">
+    <color rgba="0.75 0.75 0.75 1"/>
+  </material>
 </robot>
